File: Hardware/RTC-Messbruecke-from-template/RTC-Messbruecke-from-template.kicad_sch (KiCad schematic)
At the start: 19 parts, among them J1 Power, J2 Digital/PWM, J3 Analog, J4 Digital/PWM, J5 Conn_01x04, J6 Conn_01x04, J7 Conn_01x08, J8 Conn_01x04, U1 R-78E9.0-0.5

Commit message: modified readme
Other:
- note removed: "* Indicates a PWM-capable pin"
- company: (none) -> LMWB
- title: Template Arduino Shield Simple Outline -> 4-Fach Messbruecke PT1000
Changed lines of the file:
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@@
 	(paper "A4")
 	(title_block
-		(title "Template Arduino Shield Simple Outline")
-		(date "2024-08-05")
+		(title "4-Fach Messbruecke PT1000")
+		(date "2024-09-02")
 		(rev "v.0.2")
+		(company "LMWB")
+		(comment 1 "Lukas Bartels 2024")
 	)
 	(junction
@@
 		)
 	)
-	(text "* Indicates a PWM-capable pin"
-		(exclude_from_sim no)
-		(at 177.8 180.34 0)
-		(effects
-			(font
-				(size 1.27 1.27)
-			)
-			(justify left bottom)
-		)
-	)

Commit message: added test results and simulations
Other:
- note added: "todo - double check via dimensions! - add Modbus / CAN Tranceiver - mosfet instead of diode vor V-supply - add 5v zener diode at OP output to protect adc-input"
- note removed: "todo - double check via dimensions! - add Modbus / CAN Tranceiver - mosfet instead of diode vor V-supply"
Changed lines of the file:
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@@
 		)
 	)
-	(text "todo\n- double check via dimensions!\n- add Modbus / CAN Tranceiver\n- mosfet instead of diode vor V-supply"
+	(text "todo\n- double check via dimensions!\n- add Modbus / CAN Tranceiver\n- mosfet instead of diode vor V-supply\n- add 5v zener diode at OP output to protect adc-input"
 		(exclude_from_sim no)
-		(at 132.588 35.052 0)
+		(at 124.968 54.61 0)
 		(effects
 			(font
